Commit message: Add altimeter to urdf & simplify model

File: uuvfloat_description/urdf/uuvfloat_base.xacro (robot description, xacro)
@@ -37,16 +37,4 @@
           </geometry>
         </visual>
-        <visual name="antenna_visual">
-          <origin xyz="0 0 0" rpy=" 0 0 1.5707" />
-          <geometry>
-            <cylinder radius="0.05" length="0.3" />
-          </geometry>
-        </visual>
-        <visual name="amodem_visual">
-          <origin xyz="0 0 0" rpy=" 0 0 1.5707" />
-          <geometry>
-            <cylinder radius="0.1" length="0.3" />
-          </geometry>
-        </visual>
       </xacro:if>
       <!-- This visual geometry representation can be used when running

File: uuvfloat_description/urdf/uuvfloat_sensors.xacro (robot description, xacro)
@@ -13,37 +13,12 @@
 -->
 <robot xmlns:xacro="http://www.ros.org/wiki/xacro" >
-  <!-- DVL  -->
-  <!--
-  <xacro:default_dvl_macro
+  <!-- Altimeter  -->
+  <xacro:default_altimeter_macro
     namespace="${namespace}"
     parent_link="${namespace}/base_link"
     inertial_reference_frame="${inertial_reference_frame}">
-    <origin xyz="0.0 0.0 -0.6" rpy="0 ${0.5*pi} 0"/>
-  </xacro:default_dvl_macro>
--->
+    <origin xyz="0 0 -0.6" rpy="0 ${0.5*pi} 0"/>
+  </xacro:default_altimeter_macro>
   <!-- Magnetometer  -->
-  <xacro:default_magnetometer namespace="${namespace}" parent_link="${namespace}/base_link"/>
-  <!-- RPT  -->
-  <xacro:default_rpt namespace="${namespace}" parent_link="${namespace}/base_link">
-    <origin xyz="0 0 0.6" rpy="0 0 0"/>
-  </xacro:default_rpt>
-  <!-- Pressure  -->
-  <xacro:default_pressure_macro namespace="${namespace}" parent_link="${namespace}/base_link">
-    <origin xyz="0.0 0.0 -0.3" rpy="0 0 0"/>
-  </xacro:default_pressure_macro>
-  <!-- IMU  -->
-  <xacro:default_imu_macro
-    namespace="${namespace}"
-    parent_link="${namespace}/base_link"
-    inertial_reference_frame="${inertial_reference_frame}">
-    <origin xyz="0 0 0" rpy="0 0 0"/>
-  </xacro:default_imu_macro>
-  <!-- Mount a camera -->
-  <xacro:default_camera
-    namespace="${namespace}"
-    parent_link="${namespace}/base_link"
-    suffix="">
-    <origin xyz="0.0 0 0.0" rpy="0 0.9 0"/>
-  </xacro:default_camera>
    <!--
   <xacro:default_camera
@@ -53,24 +28,4 @@
     <origin xyz="1.15 -0.63 0.4" rpy="0 0.6 0.4"/>
   </xacro:default_camera>
-  <xacro:default_camera
-    namespace="${namespace}"
-    parent_link="${namespace}/base_link"
-    suffix="left">
-    <origin xyz="1.15 0.63 0.4" rpy="0 0.6 -0.4"/>
-  </xacro:default_camera>
 -->
-  <!-- Mount a GPS. -->
-  <xacro:default_gps namespace="${namespace}" parent_link="${namespace}/base_link" />
-  <!-- Mount a Pose 3D sensor. -->
-  <xacro:default_pose_3d_macro
-    namespace="${namespace}"
-    parent_link="${namespace}/base_link"
-    inertial_reference_frame="${inertial_reference_frame}" />
-  <!-- Mount chemical particle concentration sensor -->
-  <xacro:default_chemical_concentration_sensor_macro
-    namespace="${namespace}"
-    parent_link="${namespace}/base_link"
-    inertial_reference_frame="${inertial_reference_frame}">
-    <origin xyz="0 0 0" rpy="0 0 0"/>
-  </xacro:default_chemical_concentration_sensor_macro>
 </robot>
